File: BusSimulator.kicad_pcb (KiCad board)
At the start: 2 copper layers, 0 parts

Commit message: started 1 boost conv
Parts:
- added ARD**: Arduino_Due_Shield, BusSimulator:Arduino_Due_Shield, F.Cu at (110.0, 141.6)
- added C1: 10uF, BusSimulator:EEE-1EA100WR, F.Cu at (123.2, 130.0)
- added C2: 22uF, BusSimulator:C22, F.Cu at (127.4, 135.9)
- added C3: 10uF, BusSimulator:EEE-1EA100WR, F.Cu at (68.1, 112.3)
- added C4: 22uF, BusSimulator:EEE-1EA220WR, F.Cu at (72.0, 98.2)
- added R1: 160k, Resistors_SMD:R_0805, F.Cu at (115.0, 132.5)
- added R2: 30.1k, Resistors_SMD:R_0805, F.Cu at (115.0, 135.9)
- added R3: 100k, Resistors_SMD:R_0805, F.Cu at (118.1, 128.6)
- added R4: 63.4k, Resistors_SMD:R_0805, F.Cu at (115.4, 129.4)
- added R5: 160k, Resistors_SMD:R_0805, F.Cu at (30.4, 71.5)
- added R6: 51k, Resistors_SMD:R_0805, F.Cu at (42.1, 53.0)
- added R7: 100k, Resistors_SMD:R_0805, F.Cu at (45.4, 68.2)
- added R8: 56k, Resistors_SMD:R_0805, F.Cu at (41.7, 86.7)
- added U1: MPM3620, BusSimulator:QFN-20, F.Cu at (118.9, 134.8)
- added U2: MPM3620, BusSimulator:QFN-20, F.Cu at (75.7, 89.7)
Routing:
- net +5V: track 0.00 -> 25.3 mm, vias 0 -> 3
- net GNDA: track 0.00 -> 13.9 mm
- net GNDREF: track 0.00 -> 13.5 mm
- net (no net): track 0.00 -> 9.47 mm, vias 0 -> 6
- net Net-(C1-Pad2): track 0.00 -> 8.35 mm
- net Net-(R1-Pad2): track 0.00 -> 4.00 mm
- net Net-(R4-Pad1): track 0.00 -> 3.49 mm
- net Net-(R3-Pad2): track 0.00 -> 2.98 mm
- added copper zone on B.Cu, net +5V
- added copper zone on F.Cu, net +5V
- added copper zone on F.Cu, net GNDREF
- added copper zone on F.Cu, net Net-(C1-Pad2)
- added copper zone on F.Cu, net Net-(R1-Pad2)
