File: BusSimulator.kicad_pcb (KiCad board)
At the start: 2 copper layers, 101.6 x 53.4 mm, 100 parts, among them IC1 CS30CL, IC2 CS30CL, IC3 CS30CL, J1 CONN_3-6318491-6, J2 OSTTA024163, J3 Conn_01x03, J4 Conn_01x03, J5 Conn_01x02, J6 Conn_01x03, Q1 MOSFET_N, Q2 MOSFET_N, Q3 MOSFET_N, U1 MPM3620, U2 MPM3620, U3 MCP6H04-E/SL, U4 ADC128D818CIMTX, U5 ISO1540DR, U6 ISOInputs_Si8660_SOIC-16, U7 ISOOutputs_Si8660_SOIC-16, U8 ISOOutputs_Si8660_SOIC-16, U9 MSATA-Socket

Commit message: Organize Due-to-isolator connection
Connections:
- SHIELD1 pad 0: ISOSERO_Tx -> (no net)
- SHIELD1 pad 1: ISOSERO_Rx -> (no net)
- SHIELD1 pad 10: ISO_GPI3 -> (no net)
- SHIELD1 pad 11: ISO_GPI2 -> (no net)
- SHIELD1 pad 12: ISO_GPI1 -> (no net)
- SHIELD1 pad 13: ISO_GPI0 -> (no net)
- SHIELD1 pad 14: (no net) -> ISO_LOAD_1
- SHIELD1 pad 15: (no net) -> ISO_LOAD_2
- SHIELD1 pad 16: (no net) -> ISOSERO_Tx
- SHIELD1 pad 17: (no net) -> ISOSERO_Rx
- SHIELD1 pad 18: (no net) -> ISO_LOAD_3
- SHIELD1 pad 19: (no net) -> ISOPWRBTNn
- SHIELD1 pad 2: ISOPWR_OK -> ISOSYS_RESETn
- SHIELD1 pad 22: ISO_GPO0 -> ISO_GPI3
- SHIELD1 pad 23: ISO_GPO1 -> ISO_GPI2
- SHIELD1 pad 24: ISO_GPO2 -> ISO_GPI1
- SHIELD1 pad 25: ISO_GPO3 -> ISO_GPI0
- SHIELD1 pad 26: (no net) -> ISO_GPO3
- SHIELD1 pad 27: (no net) -> ISO_GPO2
- SHIELD1 pad 28: (no net) -> ISO_GPO1
- SHIELD1 pad 29: (no net) -> ISO_GPO0
- SHIELD1 pad 3: ISO_LOAD_3 -> (no net)
- SHIELD1 pad 4: ISO_LOAD_2 -> ISOPWR_OK
- SHIELD1 pad 5: ISO_LOAD_1 -> ISOWAKE1n
- SHIELD1 pad 6: ISO_SLEEPn -> (no net)
- SHIELD1 pad 7: ISOWAKE1n -> ISO_SLEEPn
- SHIELD1 pad 8: ISOPWRBTNn -> (no net)
- SHIELD1 pad 9: ISOSYS_RESETn -> (no net)
Routing:
- net ISO_GPI3: track 0.51 -> 0.00 mm
- net (no net): track 34.5 -> 35.0 mm
Changed lines of the file:
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@@
     (pad 21 thru_hole oval (at 86.36 -50.8) (size 1.7272 1.7272) (drill 1.016) (layers *.Cu *.Mask))
     (pad 20 thru_hole oval (at 83.82 -50.8) (size 1.7272 1.7272) (drill 1.016) (layers *.Cu *.Mask))
-    (pad 19 thru_hole oval (at 81.28 -50.8) (size 1.7272 1.7272) (drill 1.016) (layers *.Cu *.Mask))
-    (pad 18 thru_hole oval (at 78.74 -50.8) (size 1.7272 1.7272) (drill 1.016) (layers *.Cu *.Mask))
-    (pad 17 thru_hole oval (at 76.2 -50.8) (size 1.7272 1.7272) (drill 1.016) (layers *.Cu *.Mask))
-    (pad 16 thru_hole oval (at 73.66 -50.8) (size 1.7272 1.7272) (drill 1.016) (layers *.Cu *.Mask))
-    (pad 15 thru_hole oval (at 71.12 -50.8) (size 1.7272 1.7272) (drill 1.016) (layers *.Cu *.Mask))
-    (pad 14 thru_hole oval (at 68.58 -50.8) (size 1.7272 1.7272) (drill 1.016) (layers *.Cu *.Mask))
-    (pad 0 thru_hole oval (at 63.5 -50.8) (size 1.7272 1.7272) (drill 1.016) (layers *.Cu *.Mask)
+    (pad 19 thru_hole oval (at 81.28 -50.8) (size 1.7272 1.7272) (drill 1.016) (layers *.Cu *.Mask)
+      (net 96 ISOPWRBTNn))
+    (pad 18 thru_hole oval (at 78.74 -50.8) (size 1.7272 1.7272) (drill 1.016) (layers *.Cu *.Mask)
+      (net 100 ISO_LOAD_3))
+    (pad 17 thru_hole oval (at 76.2 -50.8) (size 1.7272 1.7272) (drill 1.016) (layers *.Cu *.Mask)
+      (net 94 ISOSERO_Rx))
+    (pad 16 thru_hole oval (at 73.66 -50.8) (size 1.7272 1.7272) (drill 1.016) (layers *.Cu *.Mask)
       (net 88 ISOSERO_Tx))
-    (pad 1 thru_hole oval (at 60.96 -50.8) (size 1.7272 1.7272) (drill 1.016) (layers *.Cu *.Mask)
-      (net 94 ISOSERO_Rx))
+    (pad 15 thru_hole oval (at 71.12 -50.8) (size 1.7272 1.7272) (drill 1.016) (layers *.Cu *.Mask)
+      (net 101 ISO_LOAD_2))
+    (pad 14 thru_hole oval (at 68.58 -50.8) (size 1.7272 1.7272) (drill 1.016) (layers *.Cu *.Mask)
+      (net 95 ISO_LOAD_1))
+    (pad 0 thru_hole oval (at 63.5 -50.8) (size 1.7272 1.7272) (drill 1.016) (layers *.Cu *.Mask))
+    (pad 1 thru_hole oval (at 60.96 -50.8) (size 1.7272 1.7272) (drill 1.016) (layers *.Cu *.Mask))
     (pad 2 thru_hole oval (at 58.42 -50.8) (size 1.7272 1.7272) (drill 1.016) (layers *.Cu *.Mask)
+      (net 97 ISOSYS_RESETn))
+    (pad 3 thru_hole oval (at 55.88 -50.8) (size 1.7272 1.7272) (drill 1.016) (layers *.Cu *.Mask))
+    (pad 4 thru_hole oval (at 53.34 -50.8) (size 1.7272 1.7272) (drill 1.016) (layers *.Cu *.Mask)
       (net 89 ISOPWR_OK))
-    (pad 3 thru_hole oval (at 55.88 -50.8) (size 1.7272 1.7272) (drill 1.016) (layers *.Cu *.Mask)
-      (net 100 ISO_LOAD_3))
-    (pad 4 thru_hole oval (at 53.34 -50.8) (size 1.7272 1.7272) (drill 1.016) (layers *.Cu *.Mask)
-      (net 101 ISO_LOAD_2))
     (pad 5 thru_hole oval (at 50.8 -50.8) (size 1.7272 1.7272) (drill 1.016) (layers *.Cu *.Mask)
-      (net 95 ISO_LOAD_1))
-    (pad 6 thru_hole oval (at 48.26 -50.8) (size 1.7272 1.7272) (drill 1.016) (layers *.Cu *.Mask)
+      (net 99 ISOWAKE1n))
+    (pad 6 thru_hole oval (at 48.26 -50.8) (size 1.7272 1.7272) (drill 1.016) (layers *.Cu *.Mask))
+    (pad 7 thru_hole oval (at 45.72 -50.8) (size 1.7272 1.7272) (drill 1.016) (layers *.Cu *.Mask)
       (net 98 ISO_SLEEPn))
-    (pad 7 thru_hole oval (at 45.72 -50.8) (size 1.7272 1.7272) (drill 1.016) (layers *.Cu *.Mask)
-      (net 99 ISOWAKE1n))
     (pad GND1 thru_hole oval (at 26.416 -50.8) (size 1.7272 1.7272) (drill 1.016) (layers *.Cu *.Mask)
       (net 17 GND))
-    (pad 8 thru_hole oval (at 41.656 -50.8) (size 1.7272 1.7272) (drill 1.016) (layers *.Cu *.Mask)
-      (net 96 ISOPWRBTNn))
-    (pad 9 thru_hole oval (at 39.116 -50.8) (size 1.7272 1.7272) (drill 1.016) (layers *.Cu *.Mask)
-      (net 97 ISOSYS_RESETn))
-    (pad 10 thru_hole oval (at 36.576 -50.8) (size 1.7272 1.7272) (drill 1.016) (layers *.Cu *.Mask)
-      (net 93 ISO_GPI3))
+    (pad 8 thru_hole oval (at 41.656 -50.8) (size 1.7272 1.7272) (drill 1.016) (layers *.Cu *.Mask))
+    (pad 9 thru_hole oval (at 39.116 -50.8) (size 1.7272 1.7272) (drill 1.016) (layers *.Cu *.Mask))
+    (pad 10 thru_hole oval (at 36.576 -50.8) (size 1.7272 1.7272) (drill 1.016) (layers *.Cu *.Mask))
     (pad SCL1 thru_hole oval (at 18.796 -50.8) (size 1.7272 1.7272) (drill 1.016) (layers *.Cu *.Mask)
       (net 69 DUE_SCL))
     (pad SDA1 thru_hole oval (at 21.336 -50.8) (size 1.7272 1.7272) (drill 1.016) (layers *.Cu *.Mask)
       (net 68 DUE_SDA))
-    (pad 13 thru_hole oval (at 28.956 -50.8) (size 1.7272 1.7272) (drill 1.016) (layers *.Cu *.Mask)
-      (net 90 ISO_GPI0))
-    (pad 12 thru_hole oval (at 31.496 -50.8) (size 1.7272 1.7272) (drill 1.016) (layers *.Cu *.Mask)
-      (net 91 ISO_GPI1))
-    (pad 11 thru_hole oval (at 34.036 -50.8) (size 1.7272 1.7272) (drill 1.016) (layers *.Cu *.Mask)
-      (net 92 ISO_GPI2))
+    (pad 13 thru_hole oval (at 28.956 -50.8) (size 1.7272 1.7272) (drill 1.016) (layers *.Cu *.Mask))
+    (pad 12 thru_hole oval (at 31.496 -50.8) (size 1.7272 1.7272) (drill 1.016) (layers *.Cu *.Mask))
+    (pad 11 thru_hole oval (at 34.036 -50.8) (size 1.7272 1.7272) (drill 1.016) (layers *.Cu *.Mask))
     (pad "" thru_hole oval (at 27.94 -2.54) (size 1.7272 1.7272) (drill 1.016) (layers *.Cu *.Mask))
     (pad 5V_4 thru_hole oval (at 93.98 -50.8) (size 1.7272 1.7272) (drill 1.016) (layers *.Cu *.Mask)
@@
       (net 21 "Net-(C23-Pad1)"))
     (pad 22 thru_hole oval (at 93.98 -48.26) (size 1.7272 1.7272) (drill 1.016) (layers *.Cu *.Mask)
+      (net 93 ISO_GPI3))
+    (pad 23 thru_hole oval (at 96.52 -48.26) (size 1.7272 1.7272) (drill 1.016) (layers *.Cu *.Mask)
+      (net 92 ISO_GPI2))
+    (pad 24 thru_hole oval (at 93.98 -45.72) (size 1.7272 1.7272) (drill 1.016) (layers *.Cu *.Mask)
+      (net 91 ISO_GPI1))
+    (pad 25 thru_hole oval (at 96.52 -45.72) (size 1.7272 1.7272) (drill 1.016) (layers *.Cu *.Mask)
+      (net 90 ISO_GPI0))
+    (pad 26 thru_hole oval (at 93.98 -43.18) (size 1.7272 1.7272) (drill 1.016) (layers *.Cu *.Mask)
+      (net 84 ISO_GPO3))
+    (pad 27 thru_hole oval (at 96.52 -43.18) (size 1.7272 1.7272) (drill 1.016) (layers *.Cu *.Mask)
+      (net 85 ISO_GPO2))
+    (pad 28 thru_hole oval (at 93.98 -40.64) (size 1.7272 1.7272) (drill 1.016) (layers *.Cu *.Mask)
+      (net 86 ISO_GPO1))
+    (pad 29 thru_hole oval (at 96.52 -40.64) (size 1.7272 1.7272) (drill 1.016) (layers *.Cu *.Mask)
       (net 87 ISO_GPO0))
-    (pad 23 thru_hole oval (at 96.52 -48.26) (size 1.7272 1.7272) (drill 1.016) (layers *.Cu *.Mask)
-      (net 86 ISO_GPO1))
-    (pad 24 thru_hole oval (at 93.98 -45.72) (size 1.7272 1.7272) (drill 1.016) (layers *.Cu *.Mask)
-      (net 85 ISO_GPO2))
-    (pad 25 thru_hole oval (at 96.52 -45.72) (size 1.7272 1.7272) (drill 1.016) (layers *.Cu *.Mask)
-      (net 84 ISO_GPO3))
-    (pad 26 thru_hole oval (at 93.98 -43.18) (size 1.7272 1.7272) (drill 1.016) (layers *.Cu *.Mask))
-    (pad 27 thru_hole oval (at 96.52 -43.18) (size 1.7272 1.7272) (drill 1.016) (layers *.Cu *.Mask))
-    (pad 28 thru_hole oval (at 93.98 -40.64) (size 1.7272 1.7272) (drill 1.016) (layers *.Cu *.Mask))
-    (pad 29 thru_hole oval (at 96.52 -40.64) (size 1.7272 1.7272) (drill 1.016) (layers *.Cu *.Mask))
     (pad 30 thru_hole oval (at 93.98 -38.1) (size 1.7272 1.7272) (drill 1.016) (layers *.Cu *.Mask))
     (pad 31 thru_hole oval (at 96.52 -38.1) (size 1.7272 1.7272) (drill 1.016) (layers *.Cu *.Mask))
@@
   (segment (start 121.0564 118.237) (end 121.1072 118.237) (width 0.25) (layer B.Cu) (net 0))
   (via (at 121.1072 118.237) (size 0.6) (drill 0.4) (layers F.Cu B.Cu) (net 0))
+  (segment (start 147.1168 91.4828) (end 146.759 91.125) (width 0.2) (layer B.Cu) (net 0))
   (segment (start 114.955 133.475) (end 115.855 133.475) (width 0.25) (layer F.Cu) (net 4))
   (segment (start 115.855 133.475) (end 116.11344 133.21656) (width 0.25) (layer F.Cu) (net 4))
@@
   (segment (start 125.139201 112.410801) (end 128.127199 112.410801) (width 0.2) (layer F.Cu) (net 83))
   (segment (start 120.6348 107.0864) (end 120.6348 108.3564) (width 0.2) (layer F.Cu) (net 83))
-  (segment (start 147.1168 91.4828) (end 146.759 91.125) (width 0.2) (layer B.Cu) (net 93))
   (zone (net 4) (net_name "Net-(R1-Pad2)") (layer F.Cu) (hatch edge 0.508)
     (connect_pads (clearance 0.508))
