File: BusSimulator.kicad_pcb (KiCad board)
At the start: 2 copper layers, 109.9 x 53.3 mm, 101 parts, among them IC1 CS30CL, IC2 CS30CL, IC3 CS30CL, J1 CONN_3-6318491-6, J2 OSTTA024163, J4 Conn_01x03, J5 Conn_01x02, J6 Conn_01x03, Q1 MOSFET_N, Q2 MOSFET_N, Q3 MOSFET_N, U1 MPM3620, U2 MPM3620, U3 MCP6H04-E/SL, U4 ADC128D818CIMTX, U5 ISO1540DR, U6 ISOInputs_Si8660_SOIC-16, U7 ISOOutputs_Si8660_SOIC-16, U8 ISOOutputs_Si8660_SOIC-16, U9 MSATA-Socket

Commit message: Mostly finished
Parts:
- removed C10, C23, C24, C25, C26, C30, C31: .1uF, Capacitors_SMD:C_0603
- C27, C28, C29, D1: moved to B.Cu
- moved R21 162.6 mm to (147.9, 122.4), turned to 90 degrees
- moved Q1 157.6 mm to (143.2, 112.0), turned to 90 degrees
- moved C28 150.6 mm to (158.8, 135.4), turned to 270 degrees
- moved C16 149.4 mm to (147.1, 107.6)
- moved R16 146.8 mm to (157.6, 108.9)
- moved Q2 145.8 mm to (157.6, 112.5), turned to 90 degrees
- moved R18 144.9 mm to (162.1, 122.5), turned to 90 degrees
- moved C17 143.3 mm to (161.4, 108.5)
- moved C19 139.2 mm to (149.8, 114.2), turned to 90 degrees
- moved R20 135.9 mm to (143.2, 107.8)
- moved C18 134.4 mm to (176.1, 108.2)
- moved C29 131.6 mm to (153.7, 138.3), turned to 270 degrees
- moved R13 129.5 mm to (143.4, 119.8), turned to 90 degrees
- moved C27 129.5 mm to (174.3, 137.0), turned to 90 degrees
- moved C21 127.5 mm to (179.1, 114.8), turned to 90 degrees
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Connections:
- C16 pad 1: LOAD_1 -> Load_1_PWR
- C17 pad 1: LOAD_2 -> Load_2_PWR
- C18 pad 1: LOAD_3 -> Load_3_PWR
- C29 pad 1: Net-(C29-Pad1) -> +3.3V
- IC1 pad 4: LOAD_2 -> Load_2_PWR
- IC2 pad 4: LOAD_3 -> Load_3_PWR
- IC3 pad 4: LOAD_1 -> Load_1_PWR
- J1 pad 10: Net-(J1-Pad10) -> (no net)
- J1 pad 101: Net-(J1-Pad101) -> (no net)
- J1 pad 102: Net-(J1-Pad102) -> (no net)
- J1 pad 103: Net-(J1-Pad103) -> (no net)
- J1 pad 112: Net-(J1-Pad112) -> (no net)
- J1 pad 113: Net-(J1-Pad113) -> (no net)
- J1 pad 114: Net-(J1-Pad114) -> (no net)
- J1 pad 115: Net-(J1-Pad115) -> (no net)
- J1 pad 12: Net-(J1-Pad12) -> (no net)
- J1 pad 123: Net-(J1-Pad123) -> (no net)
- J1 pad 124: Net-(J1-Pad124) -> (no net)
- J1 pad 125: Net-(J1-Pad125) -> (no net)
- J1 pad 126: Net-(J1-Pad126) -> (no net)
- J1 pad 127: Net-(J1-Pad127) -> (no net)
- J1 pad 128: Net-(J1-Pad128) -> (no net)
- J1 pad 129: Net-(J1-Pad129) -> (no net)
- J1 pad 13: Net-(J1-Pad13) -> (no net)
- J1 pad 130: Net-(J1-Pad130) -> (no net)
- J1 pad 132: Net-(J1-Pad132) -> (no net)
- J1 pad 133: Net-(J1-Pad133) -> (no net)
- J1 pad 135: Net-(J1-Pad135) -> (no net)
- J1 pad 136: Net-(J1-Pad136) -> (no net)
- J1 pad 137: Net-(J1-Pad137) -> (no net)
- J1 pad 138: Net-(J1-Pad138) -> (no net)
- J1 pad 139: Net-(J1-Pad139) -> (no net)
- J1 pad 14: Net-(J1-Pad14) -> (no net)
- J1 pad 140: Net-(J1-Pad140) -> (no net)
- J1 pad 142: Net-(J1-Pad142) -> (no net)
- J1 pad 145: Net-(J1-Pad145) -> (no net)
- J1 pad 146: Net-(J1-Pad146) -> (no net)
- J1 pad 147: Net-(J1-Pad147) -> (no net)
- J1 pad 148: Net-(J1-Pad148) -> (no net)
- J1 pad 149: Net-(J1-Pad149) -> (no net)
- J1 pad 15: Net-(J1-Pad15) -> (no net)
- J1 pad 150: Net-(J1-Pad150) -> (no net)
- J1 pad 152: Net-(J1-Pad152) -> (no net)
- J1 pad 153: Net-(J1-Pad153) -> (no net)
- J1 pad 154: Net-(J1-Pad154) -> (no net)
- J1 pad 155: Net-(J1-Pad155) -> (no net)
- J1 pad 156: Net-(J1-Pad156) -> (no net)
- J1 pad 157: Net-(J1-Pad157) -> (no net)
- J1 pad 158: Net-(J1-Pad158) -> (no net)
- J1 pad 160: Net-(J1-Pad160) -> (no net)
- J1 pad 162: Net-(J1-Pad162) -> (no net)
- J1 pad 163: Net-(J1-Pad163) -> (no net)
- J1 pad 165: Net-(J1-Pad165) -> (no net)
- J1 pad 166: Net-(J1-Pad166) -> (no net)
- J1 pad 168: Net-(J1-Pad168) -> (no net)
- J1 pad 169: Net-(J1-Pad169) -> (no net)
- J1 pad 171: Net-(J1-Pad171) -> (no net)
- J1 pad 172: Net-(J1-Pad172) -> (no net)
- J1 pad 174: Net-(J1-Pad174) -> (no net)
- J1 pad 175: Net-(J1-Pad175) -> (no net)
- J1 pad 176: Net-(J1-Pad176) -> (no net)
- J1 pad 178: Net-(J1-Pad178) -> (no net)
- J1 pad 179: Net-(J1-Pad179) -> (no net)
- J1 pad 18: Net-(J1-Pad18) -> (no net)
- J1 pad 181: Net-(J1-Pad181) -> (no net)
- J1 pad 182: Net-(J1-Pad182) -> (no net)
- J1 pad 183: Net-(J1-Pad183) -> (no net)
- J1 pad 184: Net-(J1-Pad184) -> (no net)
- J1 pad 185: Net-(J1-Pad185) -> (no net)
- J1 pad 186: Net-(J1-Pad186) -> (no net)
- J1 pad 187: Net-(J1-Pad187) -> (no net)
- J1 pad 188: Net-(J1-Pad188) -> (no net)
- J1 pad 189: Net-(J1-Pad189) -> (no net)
- J1 pad 191: Net-(J1-Pad191) -> (no net)
- J1 pad 192: Net-(J1-Pad192) -> (no net)
- J1 pad 193: Net-(J1-Pad193) -> (no net)
- J1 pad 198: Net-(J1-Pad198) -> (no net)
- J1 pad 199: Net-(J1-Pad199) -> (no net)
- J1 pad 2: Net-(J1-Pad2) -> (no net)
- J1 pad 201: Net-(J1-Pad201) -> (no net)
- J1 pad 202: Net-(J1-Pad202) -> (no net)
- J1 pad 203: Net-(J1-Pad203) -> (no net)
- J1 pad 204: Net-(J1-Pad204) -> (no net)
- J1 pad 205: Net-(J1-Pad205) -> (no net)
- J1 pad 206: Net-(J1-Pad206) -> (no net)
- J1 pad 207: Net-(J1-Pad207) -> (no net)
- J1 pad 208: Net-(J1-Pad208) -> (no net)
- J1 pad 209: Net-(J1-Pad209) -> (no net)
- J1 pad 211: Net-(J1-Pad211) -> (no net)
- J1 pad 212: Net-(J1-Pad212) -> (no net)
- J1 pad 22: Net-(J1-Pad22) -> (no net)
- J1 pad 23: Net-(J1-Pad23) -> (no net)
- J1 pad 24: Net-(J1-Pad24) -> (no net)
- J1 pad 25: Net-(J1-Pad25) -> (no net)
- J1 pad 26: Net-(J1-Pad26) -> (no net)
- J1 pad 27: Net-(J1-Pad27) -> (no net)
- J1 pad 29: Net-(J1-Pad29) -> (no net)
- J1 pad 3: Net-(J1-Pad3) -> (no net)
- J1 pad 30: Net-(J1-Pad30) -> (no net)
- J1 pad 32: Net-(J1-Pad32) -> (no net)
- J1 pad 33: Net-(J1-Pad33) -> (no net)
- J1 pad 34: Net-(J1-Pad34) -> (no net)
- J1 pad 35: Net-(J1-Pad35) -> (no net)
- J1 pad 36: Net-(J1-Pad36) -> (no net)
- J1 pad 37: Net-(J1-Pad37) -> (no net)
- J1 pad 38: Net-(J1-Pad38) -> (no net)
- J1 pad 39: Net-(J1-Pad39) -> (no net)
- J1 pad 4: Net-(J1-Pad4) -> (no net)
- J1 pad 40: Net-(J1-Pad40) -> (no net)
- J1 pad 42: Net-(J1-Pad42) -> (no net)
- J1 pad 43: Net-(J1-Pad43) -> (no net)
- J1 pad 44: Net-(J1-Pad44) -> (no net)
- J1 pad 45: Net-(J1-Pad45) -> (no net)
- J1 pad 46: Net-(J1-Pad46) -> (no net)
- J1 pad 47: Net-(J1-Pad47) -> (no net)
- J1 pad 48: Net-(J1-Pad48) -> (no net)
- J1 pad 49: Net-(J1-Pad49) -> (no net)
- J1 pad 5: Net-(J1-Pad5) -> (no net)
- J1 pad 50: Net-(J1-Pad50) -> (no net)
- J1 pad 52: Net-(J1-Pad52) -> (no net)
- J1 pad 53: Net-(J1-Pad53) -> (no net)
- J1 pad 55: Net-(J1-Pad55) -> (no net)
- J1 pad 56: Net-(J1-Pad56) -> (no net)
- J1 pad 58: Net-(J1-Pad58) -> (no net)
- J1 pad 59: Net-(J1-Pad59) -> (no net)
- J1 pad 6: Net-(J1-Pad6) -> (no net)
- J1 pad 61: Net-(J1-Pad61) -> (no net)
- J1 pad 62: Net-(J1-Pad62) -> (no net)
- J1 pad 64: Net-(J1-Pad64) -> (no net)
- J1 pad 65: Net-(J1-Pad65) -> (no net)
- J1 pad 68: Net-(J1-Pad68) -> (no net)
- J1 pad 69: Net-(J1-Pad69) -> (no net)
- J1 pad 7: Net-(J1-Pad7) -> (no net)
- J1 pad 71: Net-(J1-Pad71) -> (no net)
- J1 pad 72: Net-(J1-Pad72) -> (no net)
- J1 pad 73: Net-(J1-Pad73) -> (no net)
- J1 pad 74: Net-(J1-Pad74) -> (no net)
- J1 pad 75: Net-(J1-Pad75) -> (no net)
- J1 pad 76: Net-(J1-Pad76) -> (no net)
- J1 pad 77: Net-(J1-Pad77) -> (no net)
- J1 pad 78: Net-(J1-Pad78) -> (no net)
- J1 pad 79: Net-(J1-Pad79) -> (no net)
- J1 pad 8: Net-(J1-Pad8) -> (no net)
- J1 pad 81: Net-(J1-Pad81) -> (no net)
- J1 pad 82: Net-(J1-Pad82) -> (no net)
- J1 pad 83: Net-(J1-Pad83) -> (no net)
- J1 pad 84: Net-(J1-Pad84) -> (no net)
- J1 pad 86: Net-(J1-Pad86) -> (no net)
- J1 pad 87: Net-(J1-Pad87) -> (no net)
- J1 pad 88: Net-(J1-Pad88) -> (no net)
- J1 pad 89: Net-(J1-Pad89) -> (no net)
- J1 pad 9: Net-(J1-Pad9) -> (no net)
- J1 pad 91: Net-(J1-Pad91) -> (no net)
- J1 pad 92: Net-(J1-Pad92) -> (no net)
- J1 pad 94: Net-(J1-Pad94) -> (no net)
- J1 pad 95: Net-(J1-Pad95) -> (no net)
- J1 pad 96: Net-(J1-Pad96) -> (no net)
- J1 pad 97: Net-(J1-Pad97) -> (no net)
- Q1 pad D: LOAD_1 -> Load_1_PWR
- Q2 pad D: LOAD_2 -> Load_2_PWR
- Q3 pad D: LOAD_3 -> Load_3_PWR
- R16 pad 1: LOAD_2 -> Load_2_PWR
- R17 pad 1: LOAD_3 -> Load_3_PWR
- R20 pad 1: LOAD_1 -> Load_1_PWR
- SHIELD1 pad 10: Net-(SHIELD1-Pad10) -> (no net)
- SHIELD1 pad 11: Net-(SHIELD1-Pad11) -> (no net)
- SHIELD1 pad 12: Net-(SHIELD1-Pad12) -> (no net)
- SHIELD1 pad 13: Net-(SHIELD1-Pad13) -> (no net)
- SHIELD1 pad 20: Net-(SHIELD1-Pad20) -> (no net)
- SHIELD1 pad 21: Net-(SHIELD1-Pad21) -> (no net)
- SHIELD1 pad 3: Net-(SHIELD1-Pad3) -> (no net)
- SHIELD1 pad 30: Net-(SHIELD1-Pad30) -> (no net)
- SHIELD1 pad 31: Net-(SHIELD1-Pad31) -> (no net)
- SHIELD1 pad 32: Net-(SHIELD1-Pad32) -> (no net)
- SHIELD1 pad 33: Net-(SHIELD1-Pad33) -> (no net)
- SHIELD1 pad 34: Net-(SHIELD1-Pad34) -> (no net)
- SHIELD1 pad 35: Net-(SHIELD1-Pad35) -> (no net)
- SHIELD1 pad 5V_4: Net-(C24-Pad1) -> (no net)
- SHIELD1 pad 6: Net-(SHIELD1-Pad6) -> (no net)
- SHIELD1 pad 8: Net-(SHIELD1-Pad8) -> (no net)
- SHIELD1 pad 9: Net-(SHIELD1-Pad9) -> (no net)
- SHIELD1 pad IO_R: Net-(SHIELD1-PadIO_R) -> (no net)
- SHIELD1 pad RST: Net-(SHIELD1-PadRST) -> (no net)
- U1 pad 11: Net-(U1-Pad11) -> (no net)
- U1 pad 2: Net-(U1-Pad2) -> (no net)
- U1 pad 4: Net-(U1-Pad4) -> (no net)
- U1 pad 5: Net-(U1-Pad5) -> (no net)
- U1 pad 6: Net-(U1-Pad6) -> (no net)
- U2 pad 11: Net-(U2-Pad11) -> (no net)
- U2 pad 2: Net-(U2-Pad2) -> (no net)
- U2 pad 4: Net-(U2-Pad4) -> (no net)
- U2 pad 5: Net-(U2-Pad5) -> (no net)
- U2 pad 6: Net-(U2-Pad6) -> (no net)
- U4 pad 6: Net-(U4-Pad6) -> (no net)
- U4 pad 9: Net-(U4-Pad9) -> (no net)
- U9 pad 1: Net-(U9-Pad1) -> (no net)
- U9 pad 10: Net-(U9-Pad10) -> (no net)
- U9 pad 11: Net-(U9-Pad11) -> (no net)
- U9 pad 12: Net-(U9-Pad12) -> (no net)
- U9 pad 13: Net-(U9-Pad13) -> (no net)
- U9 pad 14: Net-(U9-Pad14) -> (no net)
- U9 pad 16: Net-(U9-Pad16) -> (no net)
- U9 pad 17: Net-(U9-Pad17) -> (no net)
- U9 pad 19: Net-(U9-Pad19) -> (no net)
- U9 pad 20: Net-(U9-Pad20) -> (no net)
- U9 pad 22: Net-(U9-Pad22) -> (no net)
- U9 pad 28: Net-(U9-Pad28) -> (no net)
- U9 pad 3: Net-(U9-Pad3) -> (no net)
- U9 pad 30: Net-(U9-Pad30) -> (no net)
- U9 pad 32: Net-(U9-Pad32) -> (no net)
- U9 pad 36: Net-(U9-Pad36) -> (no net)
- U9 pad 38: Net-(U9-Pad38) -> (no net)
- U9 pad 42: Net-(U9-Pad42) -> (no net)
- U9 pad 43: Net-(U9-Pad43) -> (no net)
- U9 pad 44: Net-(U9-Pad44) -> (no net)
- U9 pad 45: Net-(U9-Pad45) -> (no net)
- U9 pad 46: Net-(U9-Pad46) -> (no net)
- U9 pad 47: Net-(U9-Pad47) -> (no net)
- U9 pad 48: Net-(U9-Pad48) -> (no net)
- U9 pad 5: Net-(U9-Pad5) -> (no net)
- U9 pad 6: Net-(U9-Pad6) -> (no net)
- U9 pad 7: Net-(U9-Pad7) -> (no net)
- U9 pad 8: Net-(U9-Pad8) -> (no net)
Routing:
- net mCOM_GND: track 424.5 -> 602.6 mm, vias 23 -> 45
- net +3.3V: track 91.3 -> 202.5 mm, vias 14 -> 20
- net mCOM_5V_SBY: track 126.7 -> 192.9 mm, vias 12 -> 19
- net Current_3v3: track 0.00 -> 51.1 mm, vias 0 -> 1
- net LOAD_1: track 4.63 -> 53.1 mm, vias 0 -> 1
- net Current_5v: track 0.00 -> 32.9 mm, vias 0 -> 1
- net LOAD_2: track 4.76 -> 35.6 mm, vias 0 -> 1
- net LOAD_3: track 4.76 -> 26.1 mm, vias 0 -> 1
- net SATA0_TX+: track 93.5 -> 74.6 mm
- net Current_12v: track 0.00 -> 17.7 mm, vias 0 -> 1
- net Load_3_PWR: track 0.00 -> 13.1 mm
- net Load_1_PWR: track 0.00 -> 12.8 mm
- net Load_2_PWR: track 0.00 -> 12.1 mm
- net (no net): track 34.5 -> 46.4 mm, vias 2 -> 9
- net Net-(D2-Pad2): track 0.00 -> 7.95 mm
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Other:
- board text added: "12V Load"
- board text added: "3V3 Load"
- board text added: "5V Load"
