File: BusSimulator.sch (KiCad schematic (older format))
At the start: 97 parts, among them IC1 CS30CL, IC2 CS30CL, IC3 CS30CL, J1 CONN_3-6318491-6, J2 OSTTA024163, J4 Conn_01x03, J5 Conn_01x02, J6 Conn_01x03, Q1 MOSFET_N, Q2 MOSFET_N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

Commit message: finished leds
Parts:
- added D15, D16: LED, Diodes_SMD:D_1206, symbol LED
- added R33, R34: 330, Resistors_SMD:R_0603, symbol R
Connections:
- net FC3V3: no longer D10.2 (A), D11.2 (A), D12.2 (A), D13.2 (A), D14.2 (A), D9.2 (A)
- net at SHIELD1.32 (PC5): no longer R31.2
- net at SHIELD1.33 (PC4): no longer R30.2
- net at SHIELD1.34 (PC3): no longer R29.2
- net at SHIELD1.35 (PC2): no longer R28.2
- net at SHIELD1.36 (PC1): now also R34.2; no longer R27.2
- net at SHIELD1.37 (PC0): now also R33.2; no longer R26.2
- net at SHIELD1.38 (PD7): now also R31.2
- net at SHIELD1.39 (PG2): now also R30.2
- net at SHIELD1.40 (PG1): now also R29.2
- net at SHIELD1.41 (PG0): now also R28.2
- net at SHIELD1.42 (PL7): now also R27.2
- net at SHIELD1.43 (PL6): now also R26.2
- net 5V_5: now reaches C23.1, SHIELD1.5V_5
- net 5V_5: now also D10.2 (A), D11.2 (A), D12.2 (A), D13.2 (A), D14.2 (A), D9.2 (A), D15.2 (A), D16.2 (A)
- net at D9.1 (K): now also R27.1; no longer R26.1
- net at D10.1 (K): now also R26.1; no longer R27.1
- new net: D15.1 (K), R33.1
- new net: D16.1 (K), R34.1
Other:
- moved on the sheet: D10, D11, D12, D13, D14, D9, R26, R27, R28, R29, R30, R31
Changed lines of the file:
@@
 L LED D9
 U 1 1 5A0844FC
-P 15950 2150
-F 0 "D9" H 15950 2250 50  0000 C CNN
-F 1 "LED" H 15950 2050 50  0000 C CNN
-F 2 "Diodes_SMD:D_1206" H 15950 2150 50  0001 C CNN
-F 3 "" H 15950 2150 50  0001 C CNN
-	1    15950 2150
-	-1   0    0    1
+P 18750 2350
+F 0 "D9" H 18750 2450 50  0000 C CNN
+F 1 "LED" H 18750 2250 50  0000 C CNN
+F 2 "Diodes_SMD:D_1206" H 18750 2350 50  0001 C CNN
+F 3 "" H 18750 2350 50  0001 C CNN
+	1    18750 2350
+	1    0    0    -1
 $EndComp
 Text GLabel 10700 6250 0    60   Input ~ 0
@@
 Text GLabel 19000 6100 2    60   Input ~ 0
 FC5V
-Text GLabel 15800 2150 0    60   Input ~ 0
-FC3V3
+Text GLabel 18900 2350 2    60   Input ~ 0
+5V_5
 $Comp
 L LED D10
 U 1 1 5A0B9FA8
-P 15950 2250
-F 0 "D10" H 15950 2350 50  0000 C CNN
-F 1 "LED" H 15950 2150 50  0000 C CNN
-F 2 "Diodes_SMD:D_1206" H 15950 2250 50  0001 C CNN
-F 3 "" H 15950 2250 50  0001 C CNN
-	1    15950 2250
-	-1   0    0    1
+P 18750 2450
+F 0 "D10" H 18750 2550 50  0000 C CNN
+F 1 "LED" H 18750 2350 50  0000 C CNN
+F 2 "Diodes_SMD:D_1206" H 18750 2450 50  0001 C CNN
+F 3 "" H 18750 2450 50  0001 C CNN
+	1    18750 2450
+	1    0    0    -1
 $EndComp
 $Comp
 L LED D11
 U 1 1 5A0BA097
-P 15950 2350
-F 0 "D11" H 15950 2450 50  0000 C CNN
-F 1 "LED" H 15950 2250 50  0000 C CNN
-F 2 "Diodes_SMD:D_1206" H 15950 2350 50  0001 C CNN
-F 3 "" H 15950 2350 50  0001 C CNN
-	1    15950 2350
-	-1   0    0    1
+P 18750 2200
+F 0 "D11" H 18750 2300 50  0000 C CNN
+F 1 "LED" H 18750 2100 50  0000 C CNN
+F 2 "Diodes_SMD:D_1206" H 18750 2200 50  0001 C CNN
+F 3 "" H 18750 2200 50  0001 C CNN
+	1    18750 2200
+	1    0    0    -1
 $EndComp
 $Comp
 L LED D12
 U 1 1 5A0BA0A4
-P 15950 2450
-F 0 "D12" H 15950 2550 50  0000 C CNN
-F 1 "LED" H 15950 2350 50  0000 C CNN
-F 2 "Diodes_SMD:D_1206" H 15950 2450 50  0001 C CNN
-F 3 "" H 15950 2450 50  0001 C CNN
-	1    15950 2450
-	-1   0    0    1
+P 18750 2100
+F 0 "D12" H 18750 2200 50  0000 C CNN
+F 1 "LED" H 18750 2000 50  0000 C CNN
+F 2 "Diodes_SMD:D_1206" H 18750 2100 50  0001 C CNN
+F 3 "" H 18750 2100 50  0001 C CNN
+	1    18750 2100
+	1    0    0    -1
 $EndComp
 $Comp
 L LED D13
 U 1 1 5A0BA1E5
-P 15950 2550
-F 0 "D13" H 15950 2650 50  0000 C CNN
-F 1 "LED" H 15950 2450 50  0000 C CNN
-F 2 "Diodes_SMD:D_1206" H 15950 2550 50  0001 C CNN
-F 3 "" H 15950 2550 50  0001 C CNN
-	1    15950 2550
-	-1   0    0    1
+P 18750 2000
+F 0 "D13" H 18750 2100 50  0000 C CNN
+F 1 "LED" H 18750 1900 50  0000 C CNN
+F 2 "Diodes_SMD:D_1206" H 18750 2000 50  0001 C CNN
+F 3 "" H 18750 2000 50  0001 C CNN
+	1    18750 2000
+	1    0    0    -1
 $EndComp
 $Comp
 L LED D14
 U 1 1 5A0BA1F2
-P 15950 2650
-F 0 "D14" H 15950 2750 50  0000 C CNN
-F 1 "LED" H 15950 2550 50  0000 C CNN
-F 2 "Diodes_SMD:D_1206" H 15950 2650 50  0001 C CNN
-F 3 "" H 15950 2650 50  0001 C CNN
-	1    15950 2650
-	-1   0    0    1
+P 18750 1900
+F 0 "D14" H 18750 2000 50  0000 C CNN
+F 1 "LED" H 18750 1800 50  0000 C CNN
+F 2 "Diodes_SMD:D_1206" H 18750 1900 50  0001 C CNN
+F 3 "" H 18750 1900 50  0001 C CNN
+	1    18750 1900
+	1    0    0    -1
 $EndComp
 $Comp
@@
 	16400 3950 15750 3950
 Wire Wire Line
-	15450 3850 15450 3900
+	15450 3750 15450 3900
 Wire Wire Line
 	15750 4250 15750 4350
@@
 Wire Wire Line
 	7600 14150 7450 14150
-Text GLabel 15800 2250 0    60   Input ~ 0
-FC3V3
-Text GLabel 15800 2350 0    60   Input ~ 0
-FC3V3
-Text GLabel 15800 2450 0    60   Input ~ 0
-FC3V3
-Text GLabel 15800 2650 0    60   Input ~ 0
-FC3V3
-Text GLabel 15800 2550 0    60   Input ~ 0
-FC3V3
+Text GLabel 18900 2450 2    60   Input ~ 0
+5V_5
+Text GLabel 18900 2200 2    60   Input ~ 0
+5V_5
+Text GLabel 18900 2100 2    60   Input ~ 0
+5V_5
+Text GLabel 18900 1900 2    60   Input ~ 0
+5V_5
+Text GLabel 18900 2000 2    60   Input ~ 0
+5V_5
 $Comp
 L R R31
 U 1 1 5A0BA1F8
-P 16250 2650
-F 0 "R31" V 16330 2650 50  0000 C CNN
-F 1 "330" V 16250 2650 50  0000 C CNN
-F 2 "Resistors_SMD:R_0603" V 16180 2650 50  0001 C CNN
-F 3 "" H 16250 2650 50  0001 C CNN
-	1    16250 2650
-	0    -1   -1   0
+P 18450 1900
+F 0 "R31" V 18530 1900 50  0000 C CNN
+F 1 "330" V 18450 1900 50  0000 C CNN
+F 2 "Resistors_SMD:R_0603" V 18380 1900 50  0001 C CNN
+F 3 "" H 18450 1900 50  0001 C CNN
+	1    18450 1900
+	0    1    1    0
 $EndComp
 $Comp
 L R R30
 U 1 1 5A0A2423
-P 16250 2550
-F 0 "R30" V 16330 2550 50  0000 C CNN
-F 1 "330" V 16250 2550 50  0000 C CNN
-F 2 "Resistors_SMD:R_0603" V 16180 2550 50  0001 C CNN
-F 3 "" H 16250 2550 50  0001 C CNN
-	1    16250 2550
-	0    -1   -1   0
+P 18450 2000
+F 0 "R30" V 18530 2000 50  0000 C CNN
+F 1 "330" V 18450 2000 50  0000 C CNN
+F 2 "Resistors_SMD:R_0603" V 18380 2000 50  0001 C CNN
+F 3 "" H 18450 2000 50  0001 C CNN
+	1    18450 2000
+	0    1    1    0
 $EndComp
 $Comp
 L R R29
 U 1 1 5A0A2556
-P 16250 2450
-F 0 "R29" V 16330 2450 50  0000 C CNN
-F 1 "330" V 16250 2450 50  0000 C CNN
-F 2 "Resistors_SMD:R_0603" V 16180 2450 50  0001 C CNN
-F 3 "" H 16250 2450 50  0001 C CNN
-	1    16250 2450
-	0    -1   -1   0
+P 18450 2100
+F 0 "R29" V 18530 2100 50  0000 C CNN
+F 1 "330" V 18450 2100 50  0000 C CNN
+F 2 "Resistors_SMD:R_0603" V 18380 2100 50  0001 C CNN
+F 3 "" H 18450 2100 50  0001 C CNN
+	1    18450 2100
+	0    1    1    0
 $EndComp
 $Comp
 L R R28
 U 1 1 5A0A268C
-P 16250 2350
-F 0 "R28" V 16330 2350 50  0000 C CNN
-F 1 "330" V 16250 2350 50  0000 C CNN
-F 2 "Resistors_SMD:R_0603" V 16180 2350 50  0001 C CNN
-F 3 "" H 16250 2350 50  0001 C CNN
-	1    16250 2350
-	0    -1   -1   0
+P 18450 2200
+F 0 "R28" V 18530 2200 50  0000 C CNN
+F 1 "330" V 18450 2200 50  0000 C CNN
+F 2 "Resistors_SMD:R_0603" V 18380 2200 50  0001 C CNN
+F 3 "" H 18450 2200 50  0001 C CNN
+	1    18450 2200
+	0    1    1    0
 $EndComp
 $Comp
 L R R27
 U 1 1 5A0A27C5
-P 16250 2250
-F 0 "R27" V 16330 2250 50  0000 C CNN
-F 1 "330" V 16250 2250 50  0000 C CNN
-F 2 "Resistors_SMD:R_0603" V 16180 2250 50  0001 C CNN
-F 3 "" H 16250 2250 50  0001 C CNN
-	1    16250 2250
-	0    -1   -1   0
+P 18450 2350
+F 0 "R27" V 18530 2350 50  0000 C CNN
+F 1 "330" V 18450 2350 50  0000 C CNN
+F 2 "Resistors_SMD:R_0603" V 18380 2350 50  0001 C CNN
+F 3 "" H 18450 2350 50  0001 C CNN
+	1    18450 2350
+	0    1    1    0
 $EndComp
 $Comp
 L R R26
 U 1 1 5A0A2901
-P 16250 2150
-F 0 "R26" V 16330 2150 50  0000 C CNN
-F 1 "330" V 16250 2150 50  0000 C CNN
-F 2 "Resistors_SMD:R_0603" V 16180 2150 50  0001 C CNN
-F 3 "" H 16250 2150 50  0001 C CNN
-	1    16250 2150
-	0    -1   -1   0
+P 18450 2450
+F 0 "R26" V 18530 2450 50  0000 C CNN
+F 1 "330" V 18450 2450 50  0000 C CNN
+F 2 "Resistors_SMD:R_0603" V 18380 2450 50  0001 C CNN
+F 3 "" H 18450 2450 50  0001 C CNN
+	1    18450 2450
+	0    1    1    0
 $EndComp
 $Comp
@@
 Wire Wire Line
 	4250 3450 4400 3450
+$Comp
+L LED D15
+U 1 1 5A0AA4D6
+P 15950 2150
+F 0 "D15" H 15950 2250 50  0000 C CNN
+F 1 "LED" H 15950 2050 50  0000 C CNN
+F 2 "Diodes_SMD:D_1206" H 15950 2150 50  0001 C CNN
+F 3 "" H 15950 2150 50  0001 C CNN
+	1    15950 2150
+	-1   0    0    1
+$EndComp
+Text GLabel 15800 2150 0    60   Input ~ 0
+5V_5
+$Comp
+L LED D16
+U 1 1 5A0AA4DD
+P 15950 2250
+F 0 "D16" H 15950 2350 50  0000 C CNN
+F 1 "LED" H 15950 2150 50  0000 C CNN
+F 2 "Diodes_SMD:D_1206" H 15950 2250 50  0001 C CNN
+F 3 "" H 15950 2250 50  0001 C CNN
+	1    15950 2250
+	-1   0    0    1
+$EndComp
+Text GLabel 15800 2250 0    60   Input ~ 0
+5V_5
+$Comp
+L R R34
+U 1 1 5A0AA4E4
+P 16250 2250
+F 0 "R34" V 16330 2250 50  0000 C CNN
+F 1 "330" V 16250 2250 50  0000 C CNN
+F 2 "Resistors_SMD:R_0603" V 16180 2250 50  0001 C CNN
+F 3 "" H 16250 2250 50  0001 C CNN
+	1    16250 2250
+	0    -1   -1   0
+$EndComp
+$Comp
+L R R33
+U 1 1 5A0AA4EA
+P 16250 2150
+F 0 "R33" V 16330 2150 50  0000 C CNN
+F 1 "330" V 16250 2150 50  0000 C CNN
+F 2 "Resistors_SMD:R_0603" V 16180 2150 50  0001 C CNN
+F 3 "" H 16250 2150 50  0001 C CNN
+	1    16250 2150
+	0    -1   -1   0
+$EndComp
+Text GLabel 15450 3750 1    60   Input ~ 0
+5V_5
+Connection ~ 15450 3850
 $EndSCHEMATC

Commit message: Mostly finished
Parts:
- removed C10, C23, C24, C25, C26, C30, C31: .1uF, Capacitors_SMD:C_0603, symbol CAPH
Connections:
- net +3V3: now also C29.1
- net FC5V: no longer names the net of SHIELD1.5V
- net Load_1 renamed Load_1_PWR
- net Load_2 renamed Load_2_PWR
- net Load_3 renamed Load_3_PWR
Changed lines of the file:
@@
 12v_sense
 Text GLabel 8500 5700 2    60   Input ~ 0
-Load_1
+Load_1_PWR
 Text GLabel 8400 7650 2    60   Input ~ 0
 5v_sense
 Text GLabel 8500 6800 2    60   Input ~ 0
-Load_2
+Load_2_PWR
 Text GLabel 8350 8800 2    60   Input ~ 0
 3v3_sense
 Text GLabel 8450 7950 2    60   Input ~ 0
-Load_3
+Load_3_PWR
 Text GLabel 10100 1800 0    60   Input ~ 0
 Current_3v3
@@
 $EndComp
 Text GLabel 6750 11650 2    60   Input ~ 0
-Load_1
+Load_1_PWR
 $Comp
 L R R13
@@
 $EndComp
 Text GLabel 6750 12800 2    60   Input ~ 0
-Load_2
+Load_2_PWR
 $Comp
 L R R14
@@
 $EndComp
 Text GLabel 6750 13600 2    60   Input ~ 0
-Load_3
+Load_3_PWR
 $Comp
 L R R15
@@
 Text GLabel 6350 2150 0    60   Input ~ 0
 Temp
-Text GLabel 19000 6100 2    60   Input ~ 0
-FC5V
 Text GLabel 18900 2350 2    60   Input ~ 0
 5V_5
@@
 	0    1    1    0
 $EndComp
-$Comp
-L CAPH C10
-U 1 1 5A0CD143
-P 1300 14400
-F 0 "C10" H 1450 14550 60  0000 C CNN
-F 1 ".1uF" H 1450 14100 60  0000 C CNN
-F 2 "Capacitors_SMD:C_0603" H 1450 14040 60  0001 C CNN
-F 3 "" H 1300 14400 60  0000 C CNN
-	1    1300 14400
-	0    1    1    0
-$EndComp
-$Comp
-L GNDREF #PWR071
-U 1 1 5A0CD222
-P 1300 14700
-F 0 "#PWR071" H 1300 14450 50  0001 C CNN
-F 1 "GNDREF" H 1300 14550 50  0000 C CNN
-F 2 "" H 1300 14700 50  0001 C CNN
-F 3 "" H 1300 14700 50  0001 C CNN
-	1    1300 14700
-	1    0    0    -1
-$EndComp
 Text GLabel 4150 14400 2    60   Input ~ 0
 FC3V3
@@
 $EndComp
 $Comp
-L CAPH C25
-U 1 1 5A0D3367
-P 18800 6100
-F 0 "C25" H 18950 6250 60  0000 C CNN
-F 1 ".1uF" H 18950 5800 60  0000 C CNN
-F 2 "Capacitors_SMD:C_0603" H 18950 5740 60  0001 C CNN
-F 3 "" H 18800 6100 60  0000 C CNN
-	1    18800 6100
-	0    -1   -1   0
-$EndComp
-$Comp
-L CAPH C26
-U 1 1 5A0D3448
-P 18800 6200
-F 0 "C26" H 18950 6350 60  0000 C CNN
-F 1 ".1uF" H 18950 5900 60  0000 C CNN
-F 2 "Capacitors_SMD:C_0603" H 18950 5840 60  0001 C CNN
-F 3 "" H 18800 6200 60  0000 C CNN
-	1    18800 6200
-	0    1    1    0
-$EndComp
-$Comp
-L GND #PWR077
-U 1 1 5A0D39BB
-P 18800 6500
-F 0 "#PWR077" H 18800 6250 50  0001 C CNN
-F 1 "GND" H 18800 6350 50  0000 C CNN
-F 2 "" H 18800 6500 50  0001 C CNN
-F 3 "" H 18800 6500 50  0001 C CNN
-	1    18800 6500
-	1    0    0    -1
-$EndComp
-$Comp
-L GND #PWR078
-U 1 1 5A0D3A85
-P 19000 5800
-F 0 "#PWR078" H 19000 5550 50  0001 C CNN
-F 1 "GND" H 19000 5650 50  0000 C CNN
-F 2 "" H 19000 5800 50  0001 C CNN
-F 3 "" H 19000 5800 50  0001 C CNN
-	1    19000 5800
-	1    0    0    -1
-$EndComp
-$Comp
-L GND #PWR079
-U 1 1 5A0D45AE
-P 15750 4350
-F 0 "#PWR079" H 15750 4100 50  0001 C CNN
-F 1 "GND" H 15750 4200 50  0000 C CNN
-F 2 "" H 15750 4350 50  0001 C CNN
-F 3 "" H 15750 4350 50  0001 C CNN
-	1    15750 4350
-	1    0    0    -1
-$EndComp
-$Comp
-L GND #PWR080
-U 1 1 5A0D4678
-P 15450 4350
-F 0 "#PWR080" H 15450 4100 50  0001 C CNN
-F 1 "GND" H 15450 4200 50  0000 C CNN
-F 2 "" H 15450 4350 50  0001 C CNN
-F 3 "" H 15450 4350 50  0001 C CNN
-	1    15450 4350
-	1    0    0    -1
-$EndComp
-$Comp
-L CAPH C23
-U 1 1 5A0D4742
-P 15450 3900
-F 0 "C23" H 15600 4050 60  0000 C CNN
-F 1 ".1uF" H 15600 3600 60  0000 C CNN
-F 2 "Capacitors_SMD:C_0603" H 15600 3540 60  0001 C CNN
-F 3 "" H 15450 3900 60  0000 C CNN
-	1    15450 3900
-	0    1    1    0
-$EndComp
-$Comp
-L CAPH C24
-U 1 1 5A0D487F
-P 15750 3950
-F 0 "C24" H 15900 4100 60  0000 C CNN
-F 1 ".1uF" H 15900 3650 60  0000 C CNN
-F 2 "Capacitors_SMD:C_0603" H 15900 3590 60  0001 C CNN
-F 3 "" H 15750 3950 60  0000 C CNN
-	1    15750 3950
-	0    1    1    0
-$EndComp
-$Comp
 L CAPH C27
 U 1 1 5A0DCDF0
@@
 $EndComp
 $Comp
-L GNDREF #PWR081
+L GNDREF #PWR078
 U 1 1 5A0DCFAA
 P 18450 10150
-F 0 "#PWR081" H 18450 9900 50  0001 C CNN
+F 0 "#PWR078" H 18450 9900 50  0001 C CNN
 F 1 "GNDREF" H 18450 10000 50  0000 C CNN
 F 2 "" H 18450 10150 50  0001 C CNN
@@
 $EndComp
 $Comp
-L GNDREF #PWR082
+L GNDREF #PWR079
 U 1 1 5A0DD07C
 P 18800 10850
-F 0 "#PWR082" H 18800 10600 50  0001 C CNN
+F 0 "#PWR079" H 18800 10600 50  0001 C CNN
 F 1 "GNDREF" H 18800 10700 50  0000 C CNN
 F 2 "" H 18800 10850 50  0001 C CNN
 F 3 "" H 18800 10850 50  0001 C CNN
 	1    18800 10850
-	1    0    0    -1
-$EndComp
-$Comp
-L CAPH C30
-U 1 1 5A0DD40D
-P 22250 11350
-F 0 "C30" H 22400 11500 60  0000 C CNN
-F 1 ".1uF" H 22400 11050 60  0000 C CNN
-F 2 "Capacitors_SMD:C_0603" H 22400 10990 60  0001 C CNN
-F 3 "" H 22250 11350 60  0000 C CNN
-	1    22250 11350
-	0    1    1    0
-$EndComp
-$Comp
-L GNDREF #PWR083
-U 1 1 5A0DD4EC
-P 22250 11650
-F 0 "#PWR083" H 22250 11400 50  0001 C CNN
-F 1 "GNDREF" H 22250 11500 50  0000 C CNN
-F 2 "" H 22250 11650 50  0001 C CNN
-F 3 "" H 22250 11650 50  0001 C CNN
-	1    22250 11650
 	1    0    0    -1
 $EndComp
@@
 $EndComp
 $Comp
-L GNDREF #PWR084
+L GNDREF #PWR081
 U 1 1 5A0DDC34
 P 22200 10250
-F 0 "#PWR084" H 22200 10000 50  0001 C CNN
+F 0 "#PWR081" H 22200 10000 50  0001 C CNN
 F 1 "GNDREF" H 22200 10100 50  0000 C CNN
 F 2 "" H 22200 10250 50  0001 C CNN
 F 3 "" H 22200 10250 50  0001 C CNN
 	1    22200 10250
-	1    0    0    -1
-$EndComp
-$Comp
-L CAPH C31
-U 1 1 5A0DDFB1
-P 22350 12550
-F 0 "C31" H 22500 12700 60  0000 C CNN
-F 1 ".1uF" H 22500 12250 60  0000 C CNN
-F 2 "Capacitors_SMD:C_0603" H 22500 12190 60  0001 C CNN
-F 3 "" H 22350 12550 60  0000 C CNN
-	1    22350 12550
-	0    1    1    0
-$EndComp
-$Comp
-L GNDREF #PWR085
-U 1 1 5A0DE446
-P 22350 12850
-F 0 "#PWR085" H 22350 12600 50  0001 C CNN
-F 1 "GNDREF" H 22350 12700 50  0000 C CNN
-F 2 "" H 22350 12850 50  0001 C CNN
-F 3 "" H 22350 12850 50  0001 C CNN
-	1    22350 12850
 	1    0    0    -1
 $EndComp
@@
 $EndComp
 $Comp
-L GNDREF #PWR086
+L GNDREF #PWR083
 U 1 1 5A0E0BE0
 P 6100 12800
-F 0 "#PWR086" H 6100 12550 50  0001 C CNN
+F 0 "#PWR083" H 6100 12550 50  0001 C CNN
 F 1 "GNDREF" H 6100 12650 50  0000 C CNN
 F 2 "" H 6100 12800 50  0001 C CNN
@@
 $EndComp
 $Comp
-L GNDREF #PWR087
+L GNDREF #PWR084
 U 1 1 5A0E0D88
 P 6100 11650
-F 0 "#PWR087" H 6100 11400 50  0001 C CNN
+F 0 "#PWR084" H 6100 11400 50  0001 C CNN
 F 1 "GNDREF" H 6100 11500 50  0000 C CNN
 F 2 "" H 6100 11650 50  0001 C CNN
@@
 $EndComp
 $Comp
-L GNDREF #PWR088
+L GNDREF #PWR085
 U 1 1 5A0E0F30
 P 6100 13600
-F 0 "#PWR088" H 6100 13350 50  0001 C CNN
+F 0 "#PWR085" H 6100 13350 50  0001 C CNN
 F 1 "GNDREF" H 6100 13450 50  0000 C CNN
 F 2 "" H 6100 13600 50  0001 C CNN
@@
 Connection ~ 4300 1000
 Wire Wire Line
-	4500 1000 4300 1000
+	4300 1000 4500 1000
 Connection ~ 4300 5700
 Wire Wire Line
@@
 Wire Wire Line
 	1300 14400 1300 14350
-Connection ~ 1300 14400
 Wire Wire Line
 	3450 14400 4150 14400
@@
 Connection ~ 6350 2550
 Wire Wire Line
-	18300 6100 19000 6100
-Wire Wire Line
 	18300 6200 19000 6200
-Connection ~ 18800 6100
-Connection ~ 18800 6200
-Wire Wire Line
-	18800 5800 19000 5800
 Wire Wire Line
 	16400 3850 15450 3850
 Wire Wire Line
-	16400 3950 15750 3950
-Wire Wire Line
-	15450 3750 15450 3900
-Wire Wire Line
-	15750 4250 15750 4350
-Wire Wire Line
-	15450 4200 15450 4350
-Wire Wire Line
 	21150 9950 22350 9950
 Wire Wire Line
-	22350 11350 21150 11350
+	21150 11350 22350 11350
 Wire Wire Line
 	21150 12550 22450 12550
@@
 $EndComp
 $Comp
-L GNDREF #PWR089
+L GNDREF #PWR086
 U 1 1 5A0B68CF
 P 21700 9200
-F 0 "#PWR089" H 21700 8950 50  0001 C CNN
+F 0 "#PWR086" H 21700 8950 50  0001 C CNN
 F 1 "GNDREF" H 21700 9050 50  0000 C CNN
 F 2 "" H 21700 9200 50  0001 C CNN
@@
 LOAD_3
 $Comp
-L GND #PWR090
+L GND #PWR087
 U 1 1 5A0A7E15
 P 3450 15350
-F 0 "#PWR090" H 3450 15100 50  0001 C CNN
+F 0 "#PWR087" H 3450 15100 50  0001 C CNN
 F 1 "GND" H 3450 15200 50  0000 C CNN
 F 2 "" H 3450 15350 50  0001 C CNN
@@
 Text GLabel 15450 3750 1    60   Input ~ 0
 5V_5
-Connection ~ 15450 3850
+Wire Wire Line
+	15450 3850 15450 3750
+Connection ~ 22200 9950
 $EndSCHEMATC
